File: Projects/Antifurto/TILT - PIC/Tilt-PIC12F635.sch (KiCad schematic (older format))
At the start: 6 parts

Commit message: modificato Tilt-PIC12F635
Parts:
- removed C?: CAPPOL, ~, symbol CAPPOL
- removed D?: LNLED, ~, symbol LNLED
- removed P?: CONN_06, symbol CONN_06
- added C1: .01uF, ~, symbol CAP
- added DL1: LED, ~, symbol LED
- added K1: PWR, symbol CONN_03
- added K3: JAlarm, ~, symbol CONN_02
- added OC1: 4N25, DIP6, symbol 4N25
- added P1: CONN_06, ~, symbol CONN_06
- added R2: 25K, ~, symbol RESISTOR
- added R4: 33, ~, symbol RESISTOR
- added R5: 47K, ~, symbol RESISTOR
- R1: renamed from R?; value RESISTOR -> 470K
- SW1: renamed from SW?; value PULSANTENC -> TILT
- U1: renamed from U?; value PIC12F635_2 -> PIC12F635
Connections:
- net labels added: +12V, AUX, GND, ICSPCLK, ICSPDAT, Out, Tilt, VCC, VPP/MCLR
- wire segments 0 -> 43
- no-connect marks 0 -> 4
Other:
- note added: "20uA a riposo"
- note added: "Il condensatore C1 e la resistenza R2\nservono per ridurre ulteriormente il consumo.\nCon i valori indicati R=470K e C=10nF si arriva\nad un consumo di circa 70uA a riposo."
- note added: "OCT serve nel caso\ndovessi mettere \nl'accoppiatore ottico \nlontano dal uP."
- note added: "Sensore Magnetico Wi-Fi"
- moved on the sheet: R1, U1
