File: Projects/Antifurto/LampadaSirena/Lampada.sch (KiCad schematic (older format))
At the start: 5 parts

Commit message: 2014-11-19 20:41 - commit with no comment
Parts:
- gave numbers to parts that had none: 5
Connections:
- net labels added: 220Vac1, 220Vac2
- wire segments 15 -> 11
- no-connect marks 0 -> 1
Changed lines of the file:
@@
 Sheet 3 4
 Title ""
-Date "18 nov 2014"
+Date "19 nov 2014"
 Rev ""
 Comp ""
@@
 $EndDescr
 $Comp
-L RESISTOR R?
+L RESISTOR R301
 U 1 1 546AF0D6
 P 4450 3450
-F 0 "R?" V 4550 3550 40  0000 C CNN
+F 0 "R301" V 4550 3550 40  0000 C CNN
 F 1 "10K" V 4350 3550 40  0000 C CNN
 F 2 "~" H 4450 3450 60  0000 C CNN
@@
 $EndComp
 $Comp
-L VCC #PWR?
+L VCC #PWR05
 U 1 1 546AF0DC
 P 5100 2250
-F 0 "#PWR?" H 5100 2350 30  0001 C CNN
+F 0 "#PWR05" H 5100 2350 30  0001 C CNN
 F 1 "VCC" H 5100 2350 30  0000 C CNN
 F 2 "" H 5100 2250 60  0000 C CNN
@@
 $EndComp
 $Comp
-L DIODE D?
+L DIODE D301
 U 1 1 546AF0E2
 P 5100 2650
-F 0 "D?" H 5100 2750 40  0000 C CNN
+F 0 "D301" H 5100 2750 40  0000 C CNN
 F 1 "DIODE" H 5100 2550 40  0000 C CNN
 F 2 "~" H 5100 2650 60  0000 C CNN
@@
 $EndComp
 $Comp
-L NPN Q?
+L NPN Q301
 U 1 1 546AF0E8
 P 5000 3450
-F 0 "Q?" H 5000 3300 50  0000 R CNN
+F 0 "Q301" H 5000 3300 50  0000 R CNN
 F 1 "NPN" H 5000 3600 50  0000 R CNN
 F 2 "~" H 5000 3450 60  0000 C CNN
@@
 $EndComp
 $Comp
-L RELAY_1RT K?
+L RELAY_1RT K301
 U 1 1 546AF0EE
 P 4900 2700
-F 0 "K?" H 4750 2850 40  0000 C CNN
+F 0 "K301" H 4750 2850 40  0000 C CNN
 F 1 "RELAY_1RT" H 5100 2550 40  0000 C CNN
 F 2 "~" H 4900 2720 60  0000 C CNN
@@
 $EndComp
 $Comp
-L LAMP Lamp?
+L LAMP Lamp301
 U 1 1 546AF0F4
 P 4600 2350
-F 0 "Lamp?" V 4600 2550 40  0000 C CNN
+F 0 "Lamp301" V 4600 2550 40  0000 C CNN
 F 1 "LAMP" V 4400 2400 40  0000 C CNN
 F 2 "~" H 4600 2325 60  0000 C CNN
 F 3 "~" H 4600 2325 60  0000 C CNN
 	1    4600 2350
-	0    1    1    0
+	0    -1   -1   0
 $EndComp
 Text Notes 6250 2750 0    80   Italic 16
@@
 220 VAC
 $Comp
-L GNDA #PWR?
+L GNDA #PWR06
 U 1 1 546AF0FE
 P 5100 3800
-F 0 "#PWR?" H 5100 3800 40  0001 C CNN
+F 0 "#PWR06" H 5100 3800 40  0001 C CNN
 F 1 "GNDA" H 5100 3730 40  0000 C CNN
 F 2 "" H 5100 3800 60  0000 C CNN
@@
 Black (+Shield)
 Wire Wire Line
-	5100 2800 5100 2850
+	5100 2800 5100 3250
 Wire Wire Line
-	5100 2850 5100 3000
+	5100 3650 5100 3800
 Wire Wire Line
-	5100 3000 5100 3250
-Wire Wire Line
-	5100 3650 5100 3700
-Wire Wire Line
-	5100 3700 5100 3800
-Wire Wire Line
-	5100 2250 5100 2450
-Wire Wire Line
-	5100 2450 5100 2500
+	5100 2250 5100 2500
 Wire Wire Line
 	5100 3700 7000 3700
@@
 	4600 3450 4800 3450
 Wire Wire Line
-	4600 2200 4600 2100
-Wire Wire Line
-	4600 2100 3600 2100
-Wire Wire Line
 	4600 2500 4600 2650
 Wire Wire Line
 	4600 2650 4650 2650
-Wire Wire Line
-	4750 2750 3600 2750
 Connection ~ 5100 3700
 Connection ~ 5100 3000
@@
 Text HLabel 7000 3000 2    40   Output ~ 0
 LampOUT
+Text HLabel 3600 2100 0    40   Input ~ 0
+220Vac1
+Text HLabel 3600 2750 0    40   Input ~ 0
+220Vac2
+Wire Wire Line
+	3600 2750 4750 2750
+NoConn ~ 4750 2550
+Wire Wire Line
+	3600 2100 4600 2100
+Wire Wire Line
+	4600 2100 4600 2200
+Wire Bus Line
+	7500 3000 7600 3000
+Wire Bus Line
+	7600 3000 7600 3200
+Wire Bus Line
+	7600 3200 7700 3200
+Wire Bus Line
+	7700 3200 7700 3000
+Wire Bus Line
+	7700 3000 7800 3000
 $EndSCHEMATC
