File: Projects/Antifurto/LampadaSirena/LampadaSirena.sch (KiCad schematic (older format))
At the start: 23 parts, among them IC1 LTV-817, IC2 LTV-817, K1 RELAY_1RT, Q1 NPN, Q2 PNP, SW1 LampON

Commit message: 2014-11-18 07:10 - Automatic commit
Parts:
- removed D1: DIODE, ~, symbol DIODE
- removed K1: RELAY_1RT, ~, symbol RELAY_1RT
- removed Lamp1: LAMP, ~, symbol LAMP
- removed MM?: MAMMUTH10_5X2PIN, ~, symbol MAMMUTH10_5X2PIN
- removed Q1: NPN, ~, symbol NPN
- removed R1: 10K, ~, symbol RESISTOR
- removed R3: 2K7, ~, symbol RES-BOX
- removed R5: 1K, ~, symbol RES-BOX
- removed SW1, SW?: LampON, ~, symbol PULSANTENO
Connections:
- net labels added: LampON+, LampOUT+, LampOUT-, LoampON-, SirenaON
- net labels removed: +12V, VCC
- wire segments 100 -> 91
Other:
- note added: "Gray"
- note removed: "220 VAC"
- note removed: "Gray - (Sirena ON)"
- note removed: "La separazione per la doppia alimentazione è garantita dai Diodi \noppure dal Relay che viene attivato dall'alimentatore esterno.\nSi può decidere se inserire i diodi oppure il Relay. \nI diodi danno garanzia di non interruzione in caso di mancanza \ndi una delle due alimentazioni ma hanno lo svantaggio di una \ncaduta di tensione di 0,6Volt."
- note removed: "Lampada Box SENSORE"
- note removed: "Lampada \nBox 220AC"

Commit message: 2014-11-18 07:38 - Automatic commit
Connections:
- wire segments 91 -> 89
Changed lines of the file:
@@
 $Descr A4 11693 8268
 encoding utf-8
-Sheet 1 3
+Sheet 1 4
 Title ""
 Date "18 nov 2014"
@@
 $EndSheet
 Wire Wire Line
-	3350 4450 3350 2350
-Wire Wire Line
-	3350 2350 2650 2350
-Wire Wire Line
-	2650 2100 3200 2100
-Wire Wire Line
-	3200 2100 3200 4550
+	4000 2350 2650 2350
+Wire Wire Line
+	2650 2100 4000 2100
+$Sheet
+S 4000 1950 2150 800
+U 546B1B28
+F0 "SirenaBox" 50
+F1 "Sirena.sch" 50
+F2 "LampOUT" I L 4000 2100 60
+F3 "LampGND" U L 4000 2350 60
+$EndSheet
 $EndSCHEMATC

Commit message: 2014-11-18 08:06 - commit with no comment
Parts:
- removed Dev1, Dev3: ALIMENTATORE, ~, symbol ALIMENTATORE
- removed Dev2: SIRENA, ~, symbol SIRENA
- removed IC1, IC2: LTV-817, DIP4, symbol LTV-817
- removed P? (x4): CONN_04, ~, symbol CONN_04
- removed Q2: PNP, ~, symbol PNP
- removed R2: 820, ~, symbol RESISTOR
- removed R4: 2K7, ~, symbol RESISTOR
Connections:
- net labels removed: +12Vcc-A, +8V, GNDA, GO-
- wire segments 89 -> 19
Other:
- note removed: "Black (+Shield)"
- note removed: "Green/Black"
- note removed: "SIRENA - BOX"
- note removed: "Yellow"

Commit message: 2014-11-19 20:41 - commit with no comment
Parts:
- removed MM?: MAMMUTH10, ~, symbol MAMMUTH10
Connections:
- net labels removed: +12Vcc, +Batt, GND, LampON+, LampOUT+, LampOUT-, LoampON-, SirenaON
- wire segments 19 -> 2
Other:
- note removed: "Black 0.5 mm + shield"
- note removed: "Blue"
- note removed: "Gray"
- note removed: "Green"
- note removed: "Red"
- note removed: "Red 0.5 mm"
- note removed: "White"
Changed lines of the file:
@@
 Sheet 1 4
 Title ""
-Date "18 nov 2014"
+Date "19 nov 2014"
 Rev ""
 Comp ""
@@
 Comment4 ""
 $EndDescr
-Text GLabel 9250 5700 2    40   Input Italic 8
-GND
-Text GLabel 9200 5800 2    40   Input Italic 8
-+Batt
-Text Notes 8250 5800 0    40   Italic 8
-Red 0.5 mm
-$Comp
-L MAMMUTH10 MM?
-U 1 1 5451E040
-P 7600 5050
-F 0 "MM?" H 7600 5400 40  0000 C CNN
-F 1 "MAMMUTH10" H 7605 5300 40  0000 C CNN
-F 2 "~" H 7600 5050 60  0000 C CNN
-F 3 "~" H 7600 5050 60  0000 C CNN
-	1    7600 5050
-	1    0    0    -1
-$EndComp
-Wire Wire Line
-	8250 4650 8250 4650
-Wire Wire Line
-	7700 5800 9200 5800
-Wire Wire Line
-	7700 5700 9250 5700
-Wire Wire Line
-	7450 5600 7350 5600
-Wire Wire Line
-	7350 5600 7350 5700
-Wire Wire Line
-	7350 5700 7350 6000
-Wire Wire Line
-	7350 5700 7450 5700
-Wire Wire Line
-	7850 5400 7850 5500
-Wire Wire Line
-	7850 5500 7850 6250
-Wire Wire Line
-	7850 5500 7700 5500
-Connection ~ 7350 5700
-Wire Wire Line
-	7700 4900 8850 4900
-Wire Wire Line
-	7700 5100 8850 5100
-Wire Wire Line
-	7700 5000 8850 5000
-Wire Wire Line
-	7700 5200 8850 5200
-Text Notes 8250 4900 0    40   Italic 8
-White
-Text Notes 8250 5000 0    40   Italic 8
-Blue
-Text Notes 8250 5100 0    40   Italic 8
-Red
-Text Notes 8250 5200 0    40   Italic 8
-Green
-Text Notes 8250 5300 0    40   Italic 8
-Gray
-Text Notes 8250 5700 0    40   Italic 8
-Black 0.5 mm + shield
-Wire Wire Line
-	7700 5300 8850 5300
-Wire Wire Line
-	7700 5400 7850 5400
-Wire Wire Line
-	7850 5400 8900 5400
-Connection ~ 7850 5500
-Connection ~ 7850 5400
 $Sheet
 S 7100 2900 1300 1100
@@
 F7 "LampON-" U L 7100 3850 40
 $EndSheet
-Text HLabel 8850 4900 2    40   Output ~ 0
-LampOUT-
-Text HLabel 8850 5000 2    40   UnSpc ~ 0
-LampOUT+
-Text HLabel 8850 5100 2    40   Input ~ 0
-LampON+
-Text HLabel 8850 5200 2    40   UnSpc ~ 0
-LoampON-
-Text GLabel 8850 5300 2    40   Input ~ 0
-SirenaON
-Text GLabel 8900 5400 2    40   Output ~ 0
-+12Vcc
 $Sheet
 S 1250 1900 1400 700
@@
 F0 "Lampada con sensore" 50
 F1 "Lampada.sch" 50
-F2 "220Vac" I L 1250 2050 60
-F3 "220Vac" I L 1250 2250 60
+F2 "220Vac1" I L 1250 2050 60
+F3 "220Vac2" I L 1250 2250 60
 F4 "LampOUT" O R 2650 2100 60
 F5 "LampGND" U R 2650 2350 60

Commit message: 2014-11-29 09:31 - commit with no comment
Parts:
- added MM101: MAMMUTH_02A, ~, symbol MAMMUTH_02A
- added MM102: MAMMUTH_12A, ~, symbol MAMMUTH_12A
- added MM103: MAMMUTH_08A, ~, symbol MAMMUTH_08A
- added R101, R102: R, ~, symbol R
Connections:
- net labels added: +12Vcc - OUT, LampON+, LampON-, LampOUT+, LampOUT-
- wire segments 2 -> 44
Other:
- note added: "Black"
- note added: "Black 0.5 mm + shield"
- note added: "Blue"
- note added: "Gray"
- note added: "Green"
- note added: "Orange"
- note added: "Red"
- note added: "Red 0.5"
- note added: "White"
- note added: "Yellow"
- note added: "giallo-arancio-rosa-marrone"

Commit message: 2014-12-14 20:33 - commit with no comment
Parts:
- removed MM101: MAMMUTH_02A, ~, symbol MAMMUTH_02A
- removed MM102: MAMMUTH_12A, ~, symbol MAMMUTH_12A
- removed MM103: MAMMUTH_08A, ~, symbol MAMMUTH_08A
- added C101: 470uF, ~, symbol CAPPOL
- added IC101, IC102: LTV-817, DIP4, symbol LTV-817
- added MM101: MAMMUTH12, ~, symbol MAMMUTH12
- added MM102: MAMMUTH02, ~, symbol MAMMUTH02
- added MM103: MAMMUTH_08, ~, symbol MAMMUTH_08
- added R103: 1K, ~, symbol R
- added R104: 2K7, ~, symbol R
- added RXA?, RXB?, RXC?: TX-RX_4_CH, ~, symbol TX-RX_4_CH
- added SW101: DUAL_SWITCH, ~, symbol DUAL_SWITCH
- added SW102: PwrSwitch, ~, symbol DUAL_SWITCH
- R101: value R -> 27K
- R102: value R -> 56
Connections:
- net labels added: +12V, +12Vcc - IN, +Batt, -Batt, 12V-Switch, GND, LampOn+, LampOn-, SirenaON
- wire segments 44 -> 124
- no-connect marks 0 -> 7
