File: Projects/Antifurto/LampadaSirena/RadioComando.sch (KiCad schematic (older format))
At the start: 8 parts

Commit message: 2014-11-18 07:10 - Automatic commit
Connections:
- net labels added: LampON+, LampON-, LampOUT+, LampOUT-
- no-connect marks 0 -> 8
Other:
- note added: "RadioComando con 4 relay di output.\nIl primo relay (A sul telecomando) è usato \nper fare accendere la lampada manualmente. \nLo switch serve anche a disabilitare l'output di LampOUT+\nche potrebbe innescare l'antifurto e quindi la sirena. \nInfatti elimina il GND dall'emettitore del OC1 ."
Changed lines of the file:
@@
 $Descr A4 11693 8268
 encoding utf-8
-Sheet 2 2
+Sheet 2 3
 Title ""
-Date "16 nov 2014"
+Date "18 nov 2014"
 Rev ""
 Comp ""
@@
 $EndComp
 Wire Wire Line
-	2200 2450 3400 2450
-Wire Wire Line
 	2200 3100 2450 3100
 Wire Wire Line
-	2450 3100 2450 2750
-Wire Wire Line
 	2350 2900 2200 2900
 Wire Wire Line
 	2350 2650 2350 2900
 Wire Wire Line
-	2350 2650 3400 2650
-Wire Wire Line
 	2200 2650 2200 2550
-Wire Wire Line
-	2200 2550 3400 2550
-Wire Wire Line
-	2450 2750 3400 2750
 Text GLabel 5050 2850 2    40   Input ~ 0
 +12Vcc
@@
 Wire Wire Line
 	4500 2700 4500 2650
-Text GLabel 2200 3500 0    40   Input ~ 0
+Text HLabel 3200 2450 0    40   Output ~ 0
+LampON+
+Text HLabel 3200 2550 0    40   UnSpc ~ 0
+LampON-
+Text HLabel 3200 2750 0    40   Output ~ 0
+LampOUT+
+Text HLabel 3200 2650 0    40   UnSpc ~ 0
+LampOUT-
+Wire Wire Line
+	2450 3100 2450 2750
+Wire Wire Line
+	3200 2450 3400 2450
+Wire Wire Line
+	3200 2550 3400 2550
+Wire Wire Line
+	3200 2650 3400 2650
+Wire Wire Line
+	3200 2750 3400 2750
+Wire Wire Line
+	2200 2550 2750 2550
+Wire Wire Line
+	2200 2450 2750 2450
+Wire Wire Line
+	2350 2650 2750 2650
+Wire Wire Line
+	2450 2750 2750 2750
+NoConn ~ 1500 2450
+NoConn ~ 1500 2650
+NoConn ~ 1500 2900
+NoConn ~ 1500 3100
+NoConn ~ 2200 2450
+NoConn ~ 2200 2650
+NoConn ~ 2200 2900
+NoConn ~ 2200 3100
+Text HLabel 3200 2850 0    40   Input ~ 0
 +12Vcc
-Text GLabel 2200 3700 0    40   Input ~ 0
+Text HLabel 3200 2950 0    40   UnSpc ~ 0
 GND
 Wire Wire Line
-	3400 2850 2550 2850
-Wire Wire Line
-	2550 2850 2550 3500
-Wire Wire Line
-	2550 3500 2200 3500
-Wire Wire Line
-	2200 3700 2650 3700
-Wire Wire Line
-	2650 3700 2650 2950
-Wire Wire Line
-	2650 2950 3400 2950
+	3200 2850 3400 2850
+Wire Wire Line
+	3200 2950 3400 2950
+Text Notes 4450 1950 0    40   ~ 0
+RadioComando con 4 relay di output.\nIl primo relay (A sul telecomando) è usato \nper fare accendere la lampada manualmente. \nLo switch serve anche a disabilitare l'output di LampOUT+\nche potrebbe innescare l'antifurto e quindi la sirena. \nInfatti elimina il GND dall'emettitore del OC1 .
 $EndSCHEMATC

Commit message: 2014-11-19 20:41 - commit with no comment
Parts:
- removed IC? (x2): LTV-817, DIP4, symbol LTV-817
- removed MM? (x3): MAMMUTH10_5X2PIN, ~, symbol MAMMUTH10_5X2PIN
- removed R?: 2K7, ~, symbol R
- removed R?: 1K, ~, symbol R
- removed SW?: DUAL_SWITCH, ~, symbol DUAL_SWITCH
- added IC201, IC202: LTV-817, DIP4, symbol LTV-817
- added MM201: MAMMUTH10_5X2PIN, ~, symbol MAMMUTH10_5X2PIN
- added R201, R202, R204: 1K, ~, symbol R
- added R203: 2K7, ~, symbol R
- added SW201, SW202: DUAL_SWITCH, ~, symbol DUAL_SWITCH
Connections:
- net labels added: +12V, LampOn+, LampOn-, Siren-ON
- wire segments 32 -> 41
- no-connect marks 8 -> 11
Other:
- note added: "A riposo se il sensore della lampada rileva un movimento \nLo Switch serve per accendere la lampada via RadioComando.\nAcccendendo la lampada manualmente dobbiamo evitare \ndi far partire la sirena.\nQuesta è la ragione del circuito un pò più complesso.\n\nper fare accendere la lampada manualmente. \nLo switch serve anche a disabilitare l'output di LampOUT+\nche potrebbe innescare l'antifurto e q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"
- note removed: "Blue"
- note removed: "Green"
- note removed: "Red"
- note removed: "White"

Commit message: 2014-11-29 09:31 - commit with no comment
Parts:
- removed MM201: MAMMUTH10_5X2PIN, ~, symbol MAMMUTH10_5X2PIN
- removed R203: 2K7, ~, symbol R
- removed R204: 1K, ~, symbol R
- removed SW202: DUAL_SWITCH, ~, symbol DUAL_SWITCH
- added SW201, SW203: DUAL_SWITCH, ~, symbol DUAL_SWITCH
- R202: value 1K -> 2K7
- renumbered SW201 to SW202
Connections:
- net labels added: SW1-C, SW1-NC, SW1-NO, SW2-C, SW2-NC, SW2-NO
- net labels removed: LampON+, LampON-, Siren-ON
- wire segments 41 -> 28
- no-connect marks 11 -> 4

Commit message: 2014-12-14 20:33 - commit with no comment
Parts:
- added B201: DUAL_SWITCH, ~, symbol DUAL_SWITCH
- renumbered SW202 to A201, SW203 to C201
Connections:
- net labels added: A1-C, A1-NC, A1-NO, B2-C, B2-NC, B2-NO, C2-C, C2-NC, C2-NO
- net labels removed: SW1-C, SW1-NC, SW1-NO, SW2-C, SW2-NC, SW2-NO
- wire segments 28 -> 35
Changed lines of the file:
@@
 Sheet 2 4
 Title ""
-Date "26 nov 2014"
+Date "13 dec 2014"
 Rev ""
 Comp ""
@@
 Comment4 ""
 $EndDescr
-Text GLabel 6500 5250 2    40   Input ~ 0
+Text GLabel 6500 5700 2    40   Input ~ 0
 +12Vcc
-Text GLabel 6500 5350 2    40   Input ~ 0
+Text GLabel 6500 5800 2    40   Input ~ 0
 GND
 $Comp
-L DUAL_SWITCH SW202
+L DUAL_SWITCH A201
 U 1 1 546D03E6
-P 6400 5050
-F 0 "SW202" H 6700 5050 50  0000 C CNN
-F 1 "DUAL_SWITCH" H 6250 4900 50  0001 C CNN
-F 2 "~" H 6400 5050 60  0000 C CNN
-F 3 "~" H 6400 5050 60  0000 C CNN
-	1    6400 5050
+P 6400 5400
+F 0 "A201" H 6700 5400 50  0000 C CNN
+F 1 "DUAL_SWITCH" H 6250 5250 50  0001 C CNN
+F 2 "~" H 6400 5400 60  0000 C CNN
+F 3 "~" H 6400 5400 60  0000 C CNN
+	1    6400 5400
 	1    0    0    -1
 $EndComp
@@
 $EndComp
 $Comp
-L +12V #PWR01
+L +12V #PWR203
 U 1 1 5472D8CB
 P 2500 4600
-F 0 "#PWR01" H 2500 4550 20  0001 C CNN
+F 0 "#PWR203" H 2500 4550 20  0001 C CNN
 F 1 "+12V" H 2500 4700 30  0000 C CNN
 F 2 "" H 2500 4600 60  0000 C CNN
@@
 $EndComp
 $Comp
-L +12V #PWR02
+L +12V #PWR201
 U 1 1 5472D8D9
 P 2450 3100
-F 0 "#PWR02" H 2450 3050 20  0001 C CNN
+F 0 "#PWR201" H 2450 3050 20  0001 C CNN
 F 1 "+12V" H 2450 3200 30  0000 C CNN
 F 2 "" H 2450 3100 60  0000 C CNN
@@
 NoConn ~ 1400 3950
 $Comp
-L GND #PWR03
+L GND #PWR204
 U 1 1 5472D8F6
 P 2450 5750
-F 0 "#PWR03" H 2450 5750 30  0001 C CNN
+F 0 "#PWR204" H 2450 5750 30  0001 C CNN
 F 1 "GND" H 2450 5680 30  0001 C CNN
 F 2 "" H 2450 5750 60  0000 C CNN
@@
 $EndComp
 $Comp
-L GND #PWR04
+L GND #PWR202
 U 1 1 5472DA7E
 P 2650 4350
-F 0 "#PWR04" H 2650 4350 30  0001 C CNN
+F 0 "#PWR202" H 2650 4350 30  0001 C CNN
 F 1 "GND" H 2650 4280 30  0001 C CNN
 F 2 "" H 2650 4350 60  0000 C CNN
@@
 $EndComp
 $Comp
-L DUAL_SWITCH SW203
+L DUAL_SWITCH C201
 U 1 1 5472EECA
-P 6400 4750
-F 0 "SW203" H 6650 4750 50  0000 C CNN
-F 1 "DUAL_SWITCH" H 6250 4600 50  0001 C CNN
-F 2 "~" H 6400 4750 60  0000 C CNN
-F 3 "~" H 6400 4750 60  0000 C CNN
-	1    6400 4750
+P 6400 5050
+F 0 "C201" H 6650 5050 50  0000 C CNN
+F 1 "DUAL_SWITCH" H 6250 4900 50  0001 C CNN
+F 2 "~" H 6400 5050 60  0000 C CNN
+F 3 "~" H 6400 5050 60  0000 C CNN
+	1    6400 5050
 	1    0    0    -1
 $EndComp
@@
 	2100 5400 2950 5400
 Connection ~ 2500 5400
-Text HLabel 5750 5250 0    40   Input ~ 0
+Text HLabel 5750 5700 0    40   Input ~ 0
 +12Vcc
-Text HLabel 5750 5350 0    40   Input ~ 0
+Text HLabel 5750 5800 0    40   Input ~ 0
 GND
+Text HLabel 5750 5400 0    40   UnSpc ~ 0
+A1-C
+Text HLabel 5750 5500 0    40   UnSpc ~ 0
+A1-NC
+Text HLabel 5750 5300 0    40   UnSpc ~ 0
+A1-NO
+Text HLabel 5750 5150 0    40   UnSpc ~ 0
+C2-NC
 Text HLabel 5750 5050 0    40   UnSpc ~ 0
-SW1-C
-Text HLabel 5750 5150 0    40   UnSpc ~ 0
-SW1-NC
+C2-C
+Wire Wire Line
+	5750 5400 6350 5400
 Text HLabel 5750 4950 0    40   UnSpc ~ 0
-SW1-NO
-Text HLabel 5750 4850 0    40   UnSpc ~ 0
-SW2-NC
-Text HLabel 5750 4750 0    40   UnSpc ~ 0
-SW2-C
-Wire Wire Line
-	5750 5050 6350 5050
-Text HLabel 5750 4650 0    40   UnSpc ~ 0
-SW2-NO
-Wire Wire Line
-	6350 4750 5750 4750
-Wire Wire Line
-	5750 4850 6600 4850
-Wire Wire Line
-	6600 4850 6600 4800
-Wire Wire Line
-	6600 4800 6550 4800
-Wire Wire Line
-	6550 4700 6600 4700
-Wire Wire Line
-	6600 4700 6600 4650
-Wire Wire Line
-	6600 4650 5750 4650
-Wire Wire Line
-	5750 4950 6600 4950
-Wire Wire Line
-	6600 4950 6600 5000
-Wire Wire Line
-	6600 5000 6550 5000
-Wire Wire Line
-	6550 5100 6600 5100
-Wire Wire Line
-	6600 5100 6600 5150
-Wire Wire Line
-	6600 5150 5750 5150
-Wire Wire Line
-	6500 5350 5750 5350
-Wire Wire Line
-	5750 5250 6500 5250
+C2-NO
+Wire Wire Line
+	6350 5050 5750 5050
+Wire Wire Line
+	5750 5150 6600 5150
+Wire Wire Line
+	6600 5150 6600 5100
+Wire Wire Line
+	6600 5100 6550 5100
+Wire Wire Line
+	6550 5000 6600 5000
+Wire Wire Line
+	6600 5000 6600 4950
+Wire Wire Line
+	6600 4950 5750 4950
+Wire Wire Line
+	5750 5300 6600 5300
+Wire Wire Line
+	6600 5300 6600 5350
+Wire Wire Line
+	6600 5350 6550 5350
+Wire Wire Line
+	6550 5450 6600 5450
+Wire Wire Line
+	6600 5450 6600 5500
+Wire Wire Line
+	6600 5500 5750 5500
+Wire Wire Line
+	6500 5800 5750 5800
+Wire Wire Line
+	5750 5700 6500 5700
+$Comp
+L DUAL_SWITCH B201
+U 1 1 548CDF3A
+P 6400 4700
+F 0 "B201" H 6650 4700 50  0000 C CNN
+F 1 "DUAL_SWITCH" H 6250 4550 50  0001 C CNN
+F 2 "~" H 6400 4700 60  0000 C CNN
+F 3 "~" H 6400 4700 60  0000 C CNN
+	1    6400 4700
+	1    0    0    -1
+$EndComp
+Text HLabel 5750 4800 0    40   UnSpc ~ 0
+B2-NC
+Text HLabel 5750 4700 0    40   UnSpc ~ 0
+B2-C
+Text HLabel 5750 4600 0    40   UnSpc ~ 0
+B2-NO
+Wire Wire Line
+	6350 4700 5750 4700
+Wire Wire Line
+	5750 4800 6600 4800
+Wire Wire Line
+	6600 4800 6600 4750
+Wire Wire Line
+	6600 4750 6550 4750
+Wire Wire Line
+	6550 4650 6600 4650
+Wire Wire Line
+	6600 4650 6600 4600
+Wire Wire Line
+	6600 4600 5750 4600
 $EndSCHEMATC
