File: Projects/Antifurto/LampadaSirena/Sirena.sch (KiCad schematic (older format))
At the start: 13 parts

Commit message: 2014-11-18 07:38 - Automatic commit
Connections:
- net labels added: LampGND, LampOUT
Changed lines of the file:
@@
 L GNDA #PWR?
 U 1 1 546B1C67
-P 4150 3400
-F 0 "#PWR?" H 4150 3400 40  0001 C CNN
-F 1 "GNDA" H 4150 3330 40  0000 C CNN
-F 2 "" H 4150 3400 60  0000 C CNN
-F 3 "" H 4150 3400 60  0000 C CNN
-	1    4150 3400
+P 3450 3400
+F 0 "#PWR?" H 3450 3400 40  0001 C CNN
+F 1 "GNDA" H 3450 3330 40  0000 C CNN
+F 2 "" H 3450 3400 60  0000 C CNN
+F 3 "" H 3450 3400 60  0000 C CNN
+	1    3450 3400
 	1    0    0    -1
 $EndComp
@@
 L +8V #PWR?
 U 1 1 546B1C6D
-P 4150 3050
-F 0 "#PWR?" H 4150 3020 20  0001 C CNN
-F 1 "+8V" H 4150 3160 30  0000 C CNN
-F 2 "" H 4150 3050 60  0000 C CNN
-F 3 "" H 4150 3050 60  0000 C CNN
-	1    4150 3050
+P 3450 3050
+F 0 "#PWR?" H 3450 3020 20  0001 C CNN
+F 1 "+8V" H 3450 3160 30  0000 C CNN
+F 2 "" H 3450 3050 60  0000 C CNN
+F 3 "" H 3450 3050 60  0000 C CNN
+	1    3450 3050
 	1    0    0    -1
 $EndComp
@@
 	5150 3800 5150 4100
 Wire Wire Line
-	4150 3400 4150 3250
-Connection ~ 4150 3250
-Wire Wire Line
-	4150 3050 4150 3150
-Connection ~ 4150 3150
+	3450 3400 3450 3250
+Wire Wire Line
+	3450 3050 3450 3150
 Wire Wire Line
 	3300 3150 4150 3150
@@
 Connection ~ 5150 3800
 Wire Wire Line
-	3700 3800 4600 3800
-Wire Wire Line
-	3550 3900 4600 3900
+	3450 3800 4450 3800
+Wire Wire Line
+	4450 3800 4600 3800
+Wire Wire Line
+	3450 3900 4600 3900
 Wire Wire Line
 	7150 4100 7150 3650
@@
 Connection ~ 8950 5000
 Connection ~ 8950 4900
-Wire Wire Line
-	3700 3800 3700 1700
-Wire Wire Line
-	3550 1450 3550 3900
+Text HLabel 3450 3900 0    40   Input ~ 0
+LampOUT
+Text HLabel 3450 3800 0    40   UnSpc ~ 0
+LampGND
+$Comp
+L GNDA #PWR?
+U 1 1 546B2505
+P 4450 4000
+F 0 "#PWR?" H 4450 4000 40  0001 C CNN
+F 1 "GNDA" H 4450 3930 40  0000 C CNN
+F 2 "" H 4450 4000 60  0000 C CNN
+F 3 "" H 4450 4000 60  0000 C CNN
+	1    4450 4000
+	1    0    0    -1
+$EndComp
+Wire Wire Line
+	4450 3800 4450 4000
+Connection ~ 4450 3800
 $EndSCHEMATC

Commit message: 2014-11-18 08:06 - commit with no comment
Connections:
- net labels added: +Batt, LampON+, LampOUT+, LampOUT-, LoampON-, SirenaON
- wire segments 89 -> 79
Other:
- note added: "giallo-arancio-rosa-marrone"
Changed lines of the file:
@@
 	1    0    0    -1
 $EndComp
-Text Notes 9350 5300 0    40   Italic 8
+Text Notes 9300 4900 0    40   Italic 8
 Red 0.5 mm
 $Comp
@@
 Text Notes 8050 5000 0    40   Italic 8
 Yellow
-Wire Notes Line
-	9250 6350 9250 2550
 Wire Wire Line
 	3300 5850 3450 5850
@@
 	2000 4750 2150 4750
 Wire Wire Line
-	2150 4250 2150 4750
-Wire Wire Line
-	2150 4750 2150 4950
+	2150 4250 2150 4950
 Wire Wire Line
 	9350 4150 9350 4150
@@
 	5750 2750 6100 2750
 Wire Wire Line
-	5050 3900 5500 3900
-Wire Wire Line
-	5500 3900 6100 3900
+	5050 3900 6100 3900
 Wire Wire Line
 	5500 3650 5500 3900
@@
 	5150 3600 5050 3600
 Wire Wire Line
-	5150 4100 6000 4100
-Wire Wire Line
-	6000 4100 6100 4100
-Wire Wire Line
-	5150 3700 5150 3800
-Wire Wire Line
-	5150 3800 5150 4100
+	5150 4100 6100 4100
+Wire Wire Line
+	5150 3700 5150 4100
 Wire Wire Line
 	3450 3400 3450 3250
@@
 	3450 3050 3450 3150
 Wire Wire Line
-	3300 3150 4150 3150
-Wire Wire Line
-	4150 3150 4500 3150
+	3300 3150 4500 3150
 Wire Wire Line
 	4500 3150 4500 3600
@@
 	4500 3600 4600 3600
 Wire Wire Line
-	3300 3250 4150 3250
-Wire Wire Line
-	4150 3250 4400 3250
+	3300 3250 4400 3250
 Wire Wire Line
 	4400 3250 4400 3700
@@
 Connection ~ 5150 3800
 Wire Wire Line
-	3450 3800 4450 3800
-Wire Wire Line
-	4450 3800 4600 3800
+	3450 3800 4600 3800
 Wire Wire Line
 	3450 3900 4600 3900
@@
 	8800 5300 10300 5300
 Wire Wire Line
-	8800 5200 10350 5200
-Wire Wire Line
 	8550 5100 8450 5100
 Wire Wire Line
-	8450 5100 8450 5200
-Wire Wire Line
-	8450 5200 8450 5500
+	8450 5100 8450 5500
 Wire Wire Line
 	8450 5200 8550 5200
@@
 Wire Wire Line
 	8950 5750 3300 5750
-Wire Wire Line
-	8950 4900 8950 5000
 Wire Wire Line
 	8950 5000 8950 5750
@@
 Text Notes 9350 4800 0    40   Italic 8
 Gray
-Text Notes 9350 5200 0    40   Italic 8
+Text Notes 9350 5100 0    40   Italic 8
 Black 0.5 mm + shield
 Wire Wire Line
 	8800 4800 9950 4800
 Wire Wire Line
-	8800 4900 8950 4900
-Wire Wire Line
-	8950 4900 10000 4900
-Connection ~ 8950 5000
-Connection ~ 8950 4900
+	8800 4900 10000 4900
 Text HLabel 3450 3900 0    40   Input ~ 0
 LampOUT
@@
 	4450 3800 4450 4000
 Connection ~ 4450 3800
+Text GLabel 10350 5100 2    40   Input Italic 8
+GND
+Text GLabel 10300 5300 2    40   Input Italic 8
++Batt
+Text HLabel 9950 4400 2    40   Output ~ 0
+LampOUT-
+Text HLabel 9950 4500 2    40   UnSpc ~ 0
+LampOUT+
+Text HLabel 9950 4600 2    40   Input ~ 0
+LampON+
+Text HLabel 9950 4700 2    40   UnSpc ~ 0
+LoampON-
+Text GLabel 9950 4800 2    40   Input ~ 0
+SirenaON
+Text GLabel 10000 4900 2    40   Output ~ 0
++12Vcc
+Wire Wire Line
+	8800 5100 10350 5100
+Text Notes 9150 5300 0    40   Italic 8
+giallo-arancio-rosa-marrone
 $EndSCHEMATC

Commit message: 2014-11-19 20:41 - commit with no comment
Parts:
- added K401: RELAY_1RT, ~, symbol RELAY_1RT
- added MM402: MAMMUTH01, ~, symbol MAMMUTH01
- added MM403: MAMMUTH03, ~, symbol MAMMUTH03
- added MM404: MAMMUTH02, ~, symbol MAMMUTH02
- added SW401: PWR-Switch, ~, symbol PULSANTENO
- gave numbers to parts that had none: 13
Connections:
- net labels added: +12Vcc - util, +12Vcc External, +12Vcc Internal, -Batt, LampON-
- net labels removed: +12Vcc-A, LoampON-
- wire segments 79 -> 96
Other:
- note added: "Black"
- note added: "Orange"
- moved on the sheet: IC401, IC402, P401, P402, P403, P404, Q401, R401, R402

Commit message: 2014-11-29 09:31 - commit with no comment
Parts:
- removed SW401: PWR-Switch, ~, symbol PULSANTENO
- renumbered P404 to J401, P401 to J402, P403 to P401
Connections:
- net labels added: +12Vcc - IN, +12Vcc - OUT, +LampON, +LampOUT, +Lamp_IS_ON, -LampON, -LampOUT, -Lamp_IS_ON, 12V-Switch
- net labels removed: +12Vcc - util, +12Vcc External, LampGND, LampON+, LampON-, LampOUT, LampOUT+, LampOUT-
- wire segments 96 -> 95
Other:
- moved on the sheet: J401, J402, P402
Changed lines of the file:
@@
 Sheet 4 4
 Title ""
-Date "19 nov 2014"
+Date "26 nov 2014"
 Rev ""
 Comp ""
@@
 	1    0    0    -1
 $EndComp
-$Comp
-L +8V #PWR011
-U 1 1 546B1C6D
-P 3450 1700
-F 0 "#PWR011" H 3450 1670 20  0001 C CNN
-F 1 "+8V" H 3450 1810 30  0000 C CNN
-F 2 "" H 3450 1700 60  0000 C CNN
-F 3 "" H 3450 1700 60  0000 C CNN
-	1    3450 1700
-	1    0    0    -1
-$EndComp
 Text Label 2500 5300 0    40   Italic 8
 GO-
@@
 +12Vcc
 $Comp
-L CONN_04 P403
+L CONN_04 P401
 U 1 1 546B1C79
 P 4750 2500
-F 0 "P403" H 4750 2850 60  0000 C CNN
+F 0 "P401" H 4650 2950 60  0000 C CNN
 F 1 "CONN_04" H 4750 2350 60  0001 C CNN
 F 2 "~" H 4750 2500 60  0000 C CNN
@@
 $EndComp
 $Comp
-L CONN_04 P401
+L CONN_04 J402
 U 1 1 546B1C85
-P 7450 2250
-F 0 "P401" H 7450 2600 60  0000 C CNN
-F 1 "CONN_04" H 7450 2100 60  0001 C CNN
-F 2 "~" H 7450 2250 60  0000 C CNN
-F 3 "~" H 7450 2250 60  0000 C CNN
-	1    7450 2250
+P 7450 2500
+F 0 "J402" H 7350 2950 60  0000 C CNN
+F 1 "CONN_04" H 7450 2350 60  0001 C CNN
+F 2 "~" H 7450 2500 60  0000 C CNN
+F 3 "~" H 7450 2500 60  0000 C CNN
+	1    7450 2500
 	-1   0    0    -1
 $EndComp
@@
 L CONN_04 P402
 U 1 1 546B1C8B
-P 7600 2250
-F 0 "P402" H 7600 2600 60  0000 C CNN
-F 1 "CONN_04" H 7600 2100 60  0001 C CNN
-F 2 "~" H 7600 2250 60  0000 C CNN
-F 3 "~" H 7600 2250 60  0000 C CNN
-	1    7600 2250
+P 7550 2500
+F 0 "P402" H 7550 2850 60  0000 C CNN
+F 1 "CONN_04" H 7550 2350 60  0001 C CNN
+F 2 "~" H 7550 2500 60  0000 C CNN
+F 3 "~" H 7550 2500 60  0000 C CNN
+	1    7550 2500
 	1    0    0    -1
 $EndComp
@@
 L MAMMUTH10 MM401
 U 1 1 546B1C91
-P 8700 4550
-F 0 "MM401" H 8700 4900 40  0000 C CNN
-F 1 "MAMMUTH10" H 8705 4800 40  0000 C CNN
-F 2 "~" H 8700 4550 60  0000 C CNN
-F 3 "~" H 8700 4550 60  0000 C CNN
-	1    8700 4550
+P 8700 4850
+F 0 "MM401" H 8700 5550 40  0000 C CNN
+F 1 "MAMMUTH10" H 8750 5450 40  0000 C CNN
+F 2 "~" H 8700 4850 60  0000 C CNN
+F 3 "~" H 8700 4850 60  0000 C CNN
+	1    8700 4850
 	1    0    0    -1
 $EndComp
@@
 Text Notes 6850 2550 0    40   Italic 8
 Red
-Text Notes 7850 2000 0    40   Italic 8
+Text Notes 7850 2250 0    40   Italic 8
 White
-Text Notes 7850 2100 0    40   Italic 8
+Text Notes 7850 2350 0    40   Italic 8
 Blue
-Text Notes 7850 2200 0    40   Italic 8
+Text Notes 7850 2450 0    40   Italic 8
 Red
-Text Notes 7850 2300 0    40   Italic 8
+Text Notes 7850 2550 0    40   Italic 8
 Green
 Text Notes 8050 4800 0    40   Italic 8
@@
 	5750 1400 6100 1400
 Wire Wire Line
-	5050 2550 6100 2550
+	5000 2550 6100 2550
 Wire Wire Line
 	5500 2300 5500 2550
@@
 	5150 1400 5150 2250
 Wire Wire Line
-	5150 2250 5050 2250
+	5150 2250 5000 2250
 Wire Wire Line
 	5150 2750 6100 2750
@@
 	5150 2350 5150 2750
 Wire Wire Line
-	3450 2050 3450 1900
-Wire Wire Line
-	3450 1700 3450 1800
-Wire Wire Line
 	3300 1800 4500 1800
 Wire Wire Line
@@
 	4400 2350 4600 2350
 Wire Wire Line
-	5050 2350 5150 2350
+	5000 2350 5150 2350
 Wire Wire Line
 	5700 1950 5500 1950
@@
 	6800 2750 7150 2750
 Wire Wire Line
-	7100 2200 7300 2200
+	7100 2450 7300 2450
 Wire Wire Line
 	6800 2550 7100 2550
 Wire Wire Line
-	7100 1600 7100 2100
-Wire Wire Line
-	7100 2100 7300 2100
+	7100 1600 7100 2350
+Wire Wire Line
+	7100 2350 7300 2350
 Wire Wire Line
 	6800 1400 7150 1400
 Wire Wire Line
-	7150 1400 7150 2000
-Wire Wire Line
-	7150 2000 7300 2000
-Wire Wire Line
-	7100 2550 7100 2200
+	7150 1400 7150 2250
+Wire Wire Line
+	7150 2250 7300 2250
+Wire Wire Line
+	7100 2550 7100 2450
 Connection ~ 5500 2550
 Wire Wire Line
-	5050 2450 5150 2450
+	5000 2450 5150 2450
 Connection ~ 5150 2450
 Wire Wire Line
 	3450 2450 4600 2450
 Wire Wire Line
-	3450 2550 4600 2550
-Wire Wire Line
-	7150 2750 7150 2300
-Wire Wire Line
-	7150 2300 7300 2300
+	7150 2750 7150 2550
+Wire Wire Line
+	7150 2550 7300 2550
 Wire Wire Line
 	8100 4700 8550 4700
@@
 	7100 1600 6800 1600
 Wire Wire Line
-	7750 2000 8250 2000
-Wire Wire Line
-	8250 2000 8250 4400
-Wire Wire Line
-	7750 2100 8200 2100
-Wire Wire Line
-	8200 2100 8200 4500
-Wire Wire Line
-	7750 2200 8150 2200
-Wire Wire Line
-	8150 2200 8150 4600
-Wire Wire Line
-	7750 2300 8100 2300
-Wire Wire Line
-	8100 2300 8100 4700
-Wire Wire Line
-	8800 5300 10300 5300
-Wire Wire Line
-	8550 5100 8450 5100
+	7700 2250 8250 2250
+Wire Wire Line
+	8250 2250 8250 4400
+Wire Wire Line
+	7700 2350 8200 2350
+Wire Wire Line
+	8200 2350 8200 4500
+Wire Wire Line
+	7700 2450 8150 2450
+Wire Wire Line
+	8150 2450 8150 4600
+Wire Wire Line
+	7700 2550 8100 2550
+Wire Wire Line
+	8100 2550 8100 4700
+Wire Wire Line
+	8900 5300 10300 5300
 Wire Wire Line
 	8450 5100 8450 5500
@@
 Connection ~ 8450 5200
 Wire Wire Line
-	8800 4400 10200 4400
-Wire Wire Line
-	8800 4600 10200 4600
-Wire Wire Line
-	8800 4500 10200 4500
-Wire Wire Line
-	8800 4700 10200 4700
+	8900 4400 10300 4400
+Wire Wire Line
+	8900 4600 10300 4600
+Wire Wire Line
+	8900 4500 10300 4500
+Wire Wire Line
+	8900 4700 10300 4700
 Text Notes 9350 4400 0    40   Italic 8
 White
@@
 Black 0.5 mm + shield
 Wire Wire Line
-	8800 4800 10200 4800
-Wire Wire Line
-	8800 4900 10900 4900
-Text HLabel 3450 2550 0    40   Input ~ 0
-LampOUT
-Text HLabel 3450 2450 0    40   UnSpc ~ 0
-LampGND
-$Comp
-L GNDA #PWR012
+	8900 4800 10300 4800
+Wire Wire Line
+	8900 4900 10300 4900
+$Comp
+L GNDA #PWR011
 U 1 1 546B2505
 P 4450 2650
-F 0 "#PWR012" H 4450 2650 40  0001 C CNN
+F 0 "#PWR011" H 4450 2650 40  0001 C CNN
 F 1 "GNDA" H 4450 2580 40  0000 C CNN
 F 2 "" H 4450 2650 60  0000 C CNN
@@
 	4450 2450 4450 2650
 Connection ~ 4450 2450
-Text GLabel 10350 5100 2    40   Input Italic 8
-GND
-Text GLabel 10300 5300 2    40   Input Italic 8
-+Batt
-Text HLabel 10200 4400 2    40   Output ~ 0
-LampOUT-
-Text HLabel 10200 4500 2    40   UnSpc ~ 0
-LampOUT+
-Text HLabel 10200 4600 2    40   Input ~ 0
-LampON+
-Text HLabel 10200 4700 2    40   UnSpc ~ 0
-LampON-
-Text GLabel 10200 4800 2    40   Input ~ 0
-SirenaON
-Text GLabel 10250 5000 2    40   Output ~ 0
-+12Vcc - util
-Wire Wire Line
-	8800 5100 10350 5100
+Text HLabel 10300 4500 2    40   UnSpc ~ 0
+-LampOUT
+Text HLabel 10300 4400 2    40   Output ~ 0
++LampOUT
+Text HLabel 10300 4600 2    40   Input ~ 0
++LampON
+Text HLabel 10300 4700 2    40   UnSpc ~ 0
+-LampON
+Wire Wire Line
+	8900 5100 10300 5100
 Text Notes 9000 5000 0    40   Italic 8
 giallo-arancio-rosa-marrone
@@
 	-1   0    0    -1
 $EndComp
-Text GLabel 9950 5850 2    40   Input ~ 0
-+12Vcc External
-Wire Wire Line
-	10250 5000 8800 5000
-Text GLabel 10300 5200 2    40   Input Italic 8
--Batt
-Wire Wire Line
-	8800 5200 10300 5200
+Wire Wire Line
+	10300 5000 8900 5000
+Wire Wire Line
+	8900 5200 10300 5200
 Wire Wire Line
 	8550 4800 2750 4800
@@
 	2850 5500 2250 5500
 $Comp
-L CONN_04 P404
+L CONN_04 J401
 U 1 1 546B1C7F
-P 4900 2500
-F 0 "P404" H 4900 2850 60  0000 C CNN
-F 1 "CONN_04" H 4900 2350 60  0001 C CNN
-F 2 "~" H 4900 2500 60  0000 C CNN
-F 3 "~" H 4900 2500 60  0000 C CNN
-	1    4900 2500
+P 4850 2500
+F 0 "J401" H 4850 2850 60  0000 C CNN
+F 1 "CONN_04" H 4850 2350 60  0001 C CNN
+F 2 "~" H 4850 2500 60  0000 C CNN
+F 3 "~" H 4850 2500 60  0000 C CNN
+	1    4850 2500
 	1    0    0    -1
 $EndComp
 Wire Bus Line
-	2750 2500 2850 2500
+	2600 2500 2700 2500
 Wire Bus Line
-	2850 2500 2850 2650
+	2700 2500 2700 2650
 Wire Bus Line
-	2850 2650 2950 2650
+	2700 2650 2800 2650
 Wire Bus Line
-	2950 2650 2950 2500
+	2800 2650 2800 2500
 Wire Bus Line
-	2950 2500 3050 2500
+	2800 2500 2900 2500
 Text Notes 3950 1900 0    40   Italic 8
 Black (+Shield)
@@
 Text Notes 9350 4900 0    40   Italic 8
 Black
-$Comp
-L PULSANTENO SW401
-U 1 1 546CF32F
-P 10950 4950
-F 0 "SW401" V 11100 5050 50  0000 C CNN
-F 1 "PWR-Switch" V 10850 4800 40  0000 C CNN
-F 2 "~" H 10950 4950 60  0000 C CNN
-F 3 "~" H 10950 4950 60  0000 C CNN
-	1    10950 4950
-	0    1    1    0
-$EndComp
-$Comp
-L GND #PWR013
-U 1 1 546CF3CB
-P 10900 5200
-F 0 "#PWR013" H 10900 5200 30  0001 C CNN
-F 1 "GND" H 10900 5130 30  0001 C CNN
-F 2 "" H 10900 5200 60  0000 C CNN
-F 3 "" H 10900 5200 60  0000 C CNN
-	1    10900 5200
-	1    0    0    -1
-$EndComp
-Wire Wire Line
-	10900 5000 10900 5200
 Wire Notes Line
 	3150 6500 4150 6500
@@
 Wire Notes Line
 	3150 7450 3150 6500
+Wire Wire Line
+	8550 5100 8450 5100
+Wire Wire Line
+	4600 2550 3450 2550
+$Comp
+L +8V #PWR012
+U 1 1 5472EB2B
+P 3450 1650
+F 0 "#PWR012" H 3450 1620 20  0001 C CNN
+F 1 "+8V" H 3450 1760 30  0000 C CNN
+F 2 "" H 3450 1650 60  0000 C CNN
+F 3 "" H 3450 1650 60  0000 C CNN
+	1    3450 1650
+	1    0    0    -1
+$EndComp
+Wire Wire Line
+	3450 1650 3450 1800
+Connection ~ 3450 1800
+Connection ~ 3450 1900
+Wire Wire Line
+	3450 2050 3450 1900
+Text HLabel 10300 4800 2    40   UnSpc ~ 0
+SirenaON
+Text HLabel 10300 5300 2    40   Input ~ 0
++Batt
+Text HLabel 10300 5200 2    40   UnSpc ~ 0
+-Batt
+Text HLabel 10300 5100 2    40   UnSpc ~ 0
+GND
+Text HLabel 10300 5000 2    40   Output ~ 0
++12Vcc - OUT
+Text HLabel 10300 4900 2    40   UnSpc ~ 0
+12V-Switch
+Text HLabel 9950 5850 2    40   Input ~ 0
++12Vcc - IN
+Text HLabel 3450 2450 0    40   UnSpc ~ 0
+-Lamp_IS_ON
+Text HLabel 3450 2550 0    40   Output ~ 0
++Lamp_IS_ON
 $EndSCHEMATC

Commit message: 2014-12-14 20:33 - commit with no comment
Changed lines of the file:
@@
 Sheet 4 4
 Title ""
-Date "26 nov 2014"
+Date "13 dec 2014"
 Rev ""
 Comp ""
@@
 $EndComp
 $Comp
-L GND #PWR07
+L GND #PWR406
 U 1 1 546B1C35
 P 2400 6300
-F 0 "#PWR07" H 2400 6300 30  0001 C CNN
+F 0 "#PWR406" H 2400 6300 30  0001 C CNN
 F 1 "GND" H 2400 6230 30  0001 C CNN
 F 2 "" H 2400 6300 60  0000 C CNN
@@
 $EndComp
 $Comp
-L GND #PWR08
+L GND #PWR405
 U 1 1 546B1C3B
 P 2400 5800
-F 0 "#PWR08" H 2400 5800 30  0001 C CNN
+F 0 "#PWR405" H 2400 5800 30  0001 C CNN
 F 1 "GND" H 2400 5730 30  0001 C CNN
 F 2 "" H 2400 5800 60  0000 C CNN
@@
 Red 0.5 mm
 $Comp
-L GND #PWR09
+L GND #PWR404
 U 1 1 546B1C42
 P 8450 5500
-F 0 "#PWR09" H 8450 5500 30  0001 C CNN
+F 0 "#PWR404" H 8450 5500 30  0001 C CNN
 F 1 "GND" H 8450 5430 30  0001 C CNN
 F 2 "" H 8450 5500 60  0000 C CNN
@@
 $EndComp
 $Comp
-L GNDA #PWR010
+L GNDA #PWR402
 U 1 1 546B1C67
 P 3450 2050
-F 0 "#PWR010" H 3450 2050 40  0001 C CNN
+F 0 "#PWR402" H 3450 2050 40  0001 C CNN
 F 1 "GNDA" H 3450 1980 40  0000 C CNN
 F 2 "" H 3450 2050 60  0000 C CNN
@@
 	8900 4900 10300 4900
 $Comp
-L GNDA #PWR011
+L GNDA #PWR403
 U 1 1 546B2505
 P 4450 2650
-F 0 "#PWR011" H 4450 2650 40  0001 C CNN
+F 0 "#PWR403" H 4450 2650 40  0001 C CNN
 F 1 "GNDA" H 4450 2580 40  0000 C CNN
 F 2 "" H 4450 2650 60  0000 C CNN
@@
 L MAMMUTH02 MM404
 U 1 1 546CEB55
-P 4100 6550
-F 0 "MM404" H 4100 6900 40  0001 C CNN
-F 1 "MAMMUTH02" H 4105 6800 40  0001 C CNN
-F 2 "~" H 4100 6550 60  0000 C CNN
-F 3 "~" H 4100 6550 60  0000 C CNN
-	1    4100 6550
+P 3950 6700
+F 0 "MM404" H 3950 7050 40  0001 C CNN
+F 1 "MAMMUTH02" H 3955 6950 40  0001 C CNN
+F 2 "~" H 3950 6700 60  0000 C CNN
+F 3 "~" H 3950 6700 60  0000 C CNN
+	1    3950 6700
 	0    -1   -1   0
 $EndComp
@@
 	4600 2550 3450 2550
 $Comp
-L +8V #PWR012
+L +8V #PWR401
 U 1 1 5472EB2B
 P 3450 1650
-F 0 "#PWR012" H 3450 1620 20  0001 C CNN
+F 0 "#PWR401" H 3450 1620 20  0001 C CNN
 F 1 "+8V" H 3450 1760 30  0000 C CNN
 F 2 "" H 3450 1650 60  0000 C CNN
