File: Projects/Timer4Autoradio/Timer4Autoradio-PIC12F635.kicad_pcb (KiCad board)
At the start: 2 copper layers, 21 parts, among them IC1 4N35, K1 12Vcc, K3 RELAY_1RT, P1 CONN_06, SW1 Power, U1 78L05, U2 PIC12F635

Commit message: 2014-11-30 21:10 - commit with no comment
Parts:
- C2: footprint C1V5 -> CAPE_100_V5
- R1, R2, R3, R4, R5: footprint R5 -> Res-500
- U1: footprint LM78XX-TO92 -> LM78XX-TO92-ELL
- U2: footprint Ln_DIP-8_300 -> DIP-8_300
- moved K3 120.3 mm to (163.8, 67.3)
- moved R1 106.0 mm to (151.1, 104.1)
- moved C3 90.6 mm to (77.5, 111.8), turned to 270 degrees
- moved IC1 88.2 mm to (55.9, 124.5), turned to 270 degrees
- moved K1 87.8 mm to (34.3, 105.4)
- moved U2 85.7 mm to (41.9, 125.7), turned to 270 degrees
- moved DL1 75.1 mm to (125.7, 111.8)
- moved DL3 73.4 mm to (49.5, 87.6)
- moved D1 61.3 mm to (48.3, 108.0)
- moved C1 59.9 mm to (59.7, 109.2), turned to 270 degrees
- moved SW1 49.8 mm to (71.1, 72.4)
- moved R3 48.1 mm to (129.5, 45.7)
- moved R5 47.0 mm to (43.2, 80.0), turned to 90 degrees
- moved R2 43.4 mm to (63.5, 47.0)
- moved U1 42.7 mm to (68.6, 110.5), turned to 90 degrees
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
Commit message: 2015-02-06 07:53 - commit with no comment
Parts:
- removed D4: DIODE, Diode_500
- removed DL3: LED, LED-5MM
- removed K1: 12Vcc, SIP-03
- removed K3: RELAY_1RT, DIP-14_300
- removed P1: CONN_06, SIP-06
- removed SW1: Power, SIP-03
- added C4: 10uF, LnCAPE_100_V5, F.Cu at (78.7, 35.6)
- added J1: 12Vcc, LnSIP-04, F.Cu at (114.3, 43.2)
- added J2: ExtLED, LnSIP-02, F.Cu at (114.3, 68.6)
- added J3: CONN_05, LnSIP-05, F.Cu at (66.0, 76.2)
- added PB1: PButton, LnSIP-02, F.Cu at (114.3, 76.2)
- added Q1: BC337-BC238, Ln-TO92-BC238, F.Cu at (76.2, 43.2)
- added R6: 470, LnRes-500, F.Cu at (73.7, 58.4)
- added R7: 2k2, LnRes-500, F.Cu at (86.4, 30.5)
- added RL1: RELAY_AUTORADIO, LnDIP-14_300, F.Cu at (88.9, 35.6)
- C1, C3: value C -> 100nF; footprint Cap_100 -> LnCap_100
- C2: value CAPPOL -> 10uF; footprint CAPE_100_V5 -> LnCAPE_100_V5
- D1, D2: footprint Diode_500 -> LnDiode_500
- DL1, DL2: footprint LED-5MM -> LnLED-5MM
- IC1: footprint DIP-6_300 -> LnDIP-06_300
- R1: value 27K -> 25K; footprint Res-500 -> LnRes-500
- R2: value 100K -> 4K7; footprint Res-500 -> LnRes-500
- R3: value 25K -> 2K2; footprint Res-500 -> LnRes-500
- R4: value 470 -> 25K; footprint Res-500 -> LnRes-500
- R5: value 470K -> 330; footprint Res-500 -> LnRes-500
- U1: footprint LM78XX-TO92-ELL -> LnLM78XX-TO92
- U2: value PIC12F635 -> PIC12F635_4; footprint DIP-8_300 -> LnDIP-08_300
- moved D1 98.6 mm to (109.2, 30.5), turned to 180 degrees
- moved DL1 85.4 mm to (68.6, 48.3), turned to 180 degrees
- moved IC1 78.4 mm to (88.9, 53.3), turned to 0 degrees
- moved C1 78.0 mm to (109.9, 49.5)
- moved U2 74.0 mm to (88.9, 68.6), turned to 0 degrees
- moved R1 72.8 mm to (101.6, 50.8), turned to 90 degrees
- moved U1 63.1 mm to (104.1, 58.4)
- moved C2 62.1 mm to (109.9, 58.4), turned to 0 degrees
- moved R3 61.0 mm to (68.6, 43.2), turned to 90 degrees
- moved C3 58.1 mm to (109.9, 63.5), turned to 0 degrees
- moved R4 47.4 mm to (83.8, 63.5)
- moved R2 44.1 mm to (106.7, 38.1), turned to 270 degrees
- moved D2 42.7 mm to (83.8, 41.9)
- moved R5 36.1 mm to (78.7, 73.7)
- moved DL2 27.9 mm to (68.6, 55.9), turned to 180 degrees
Connections:
- C1 pad 1: N-0000010 (its old number) -> /+12Vcc (Autoradio)
- C3 pad 1: N-000009 -> +5V
- D1 pad 2: N-0000010 (its old number) -> N-0000014
- D2 pad 1: N-000009 -> N-0000012
- D2 pad 2: +5V -> N-0000014
- DL1 pad 1: +12V -> N-000003
- DL1 pad 2: N-000007 -> N-000004
- DL2 pad 1: N-000002 -> N-000009
- DL2 pad 2: N-000001 -> GND
- IC1 pad 1: N-000001 -> N-000004
- IC1 pad 5: N-000007 -> N-0000012
- IC1 pad 6: N-0000012 -> (no net)
- R1 pad 1: N-0000011 -> /+12V_CMD
- R1 pad 2: N-0000012 -> N-0000013
- R2 pad 1: N-0000012 -> /+12V_CMD
- R2 pad 2: GND -> ICSPDAT
- R3 pad 1: +5V -> ICSPDAT
- R3 pad 2: VPP/MCLR -> GND
- R4 pad 1: N-000002 -> +5V
- R4 pad 2: /Out -> VPP/MCLR
- R5 pad 1: N-0000023 -> /ClockOUT
- R5 pad 2: N-0000018 -> N-000003
- U1 pad VI: N-0000010 (its old number) -> /+12Vcc (Autoradio)
- U1 pad VO: N-000009 -> +5V
- U2 pad 2: N-0000018 -> N-000002
- U2 pad 3: /Out -> /ClockOUT
Routing:
- net GND: track 0.00 -> 163.4 mm
- net ICSPDAT: track 0.00 -> 102.1 mm, vias 0 -> 2
- net /+12Vcc (Autoradio): track 0.00 -> 73.9 mm, vias 0 -> 2
- net +5V: track 0.00 -> 71.4 mm
- net N-0000012: track 0.00 -> 62.2 mm
- net N-000009: track 0.00 -> 55.0 mm
- net ICSPCLK: track 0.00 -> 45.9 mm
- net N-0000014: track 0.00 -> 44.0 mm
- net N-0000013: track 0.00 -> 30.5 mm, vias 0 -> 2
- net /+12V_CMD: track 0.00 -> 30.0 mm
- net N-000004: track 0.00 -> 27.6 mm, vias 0 -> 2
- net VPP/MCLR: track 0.00 -> 22.9 mm
- net N-0000011: track 0.00 -> 20.6 mm
- net N-000003: track 0.00 -> 18.4 mm
- net N-0000010: track 0.00 -> 17.8 mm
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Other:
- copper layers 2 -> 6
