File: Projects/Timer4Autoradio/Timer4Autoradio-PIC12F635.sch (KiCad schematic (older format))
At the start: 10 parts, among them K1 PWR, P1 CONN_06, SW1 Power, U1 PIC12F635

Commit message: 2014-11-29 09:31 - commit with no comment
Parts:
- added DL1: LED, ~, symbol LED
- added R4: 470K, ~, symbol RESISTOR
- gave numbers to parts that had none: 5
- renumbered R2 to R1
Connections:
- wire segments 40 -> 37
- no-connect marks 3 -> 5
Other:
- moved on the sheet: D1, K1, K2, Q1, R2, R3

Commit message: 2014-11-29 21:44 - commit with no comment
Parts:
- removed K2: RELAY_1RT, ~, symbol RELAY_1RT
- removed Q1: NPN, ~, symbol NPN
- removed R3: 470K, ~, symbol RESISTOR
- added C1, C3: C, ~, symbol C
- added C2: CAPPOL, ~, symbol CAPPOL
- added D2: 1N4148, ~, symbol DIODE
- added D4: DIODE, ~, symbol DIODE
- added DL1, DL2: LED, ~, symbol LED
- added IC1: 4N35, ~, symbol 4N35
- added K3: RELAY_1RT, ~, symbol RELAY_1RT
- added R1: 27K, ~, symbol RESISTOR
- added R2: 100K, ~, symbol RESISTOR
- added U1: 78L05, ~, symbol 78L05
- D1: value DIODE -> 1N4001
- K1: value PWR -> 12Vcc
- R4: renamed from R2; value 470K -> 470
- U2: renamed from U1; footprint ~ -> Ln_DIP-8_300
- renumbered DL1 to DL3, R1 to R3, R4 to R5
Connections:
- net labels added: +5V
- wire segments 37 -> 65
- no-connect marks 5 -> 4
Other:
- note added: "12Vcc comandata"
- moved on the sheet: DL3, K1, R3, R4, R5, U2

Commit message: 2014-11-30 21:10 - commit with no comment
Parts:
- removed U2: PIC12F635, Ln_DIP-8_300, symbol PIC12F635_2
- added U2: PIC12F635, ~, symbol PIC12F635_3
- K1: footprint (none) -> ~
Connections:
- wire segments 65 -> 63
Other:
- moved on the sheet: R1, R2
Changed lines of the file:
@@
 EESchema Schematic File Version 2
+LIBS:LnRegulators
 LIBS:Ln_R-C-L
 LIBS:LnConnectors
@@
 Sheet 1 1
 Title "Tilt per antifurto con PIC12F635"
-Date "29 nov 2014"
+Date "30 nov 2014"
 Rev "0.5"
 Comp "Loreto N."
@@
 Comment4 ""
 $EndDescr
-$Comp
-L PIC12F635_2 U2
-U 1 1 53664521
-P 4750 5950
-F 0 "U2" H 4500 6800 60  0000 C CNN
-F 1 "PIC12F635" H 5100 6800 60  0000 C CNN
-F 2 "Ln_DIP-8_300" H 5150 5750 60  0000 C CNN
-F 3 "~" H 4750 5950 60  0000 C CNN
-	1    4750 5950
-	1    0    0    -1
-$EndComp
 $Comp
 L PULSANTENC SW1
@@
 F 0 "K1" H 1400 3700 50  0000 C CNN
 F 1 "12Vcc" H 1400 3600 40  0000 C CNN
-F 2 "" H 1600 3450 60  0000 C CNN
+F 2 "~" H 1600 3450 60  0000 C CNN
 F 3 "" H 1600 3450 60  0000 C CNN
 	1    1600 3450
@@
 $EndComp
 $Comp
-L VCC #PWR01
+L VCC #PWR1
 U 1 1 53994E0E
 P 4000 1550
-F 0 "#PWR01" H 4000 1650 30  0001 C CNN
+F 0 "#PWR1" H 4000 1650 30  0001 C CNN
 F 1 "VCC" H 4000 1650 30  0000 C CNN
 F 2 "" H 4000 1550 60  0000 C CNN
@@
 $EndComp
 $Comp
-L GND #PWR02
+L GND #PWR16
 U 1 1 53994E1D
 P 4750 6450
-F 0 "#PWR02" H 4750 6450 30  0001 C CNN
+F 0 "#PWR16" H 4750 6450 30  0001 C CNN
 F 1 "GND" H 4750 6380 30  0001 C CNN
 F 2 "" H 4750 6450 60  0000 C CNN
@@
 $EndComp
 $Comp
-L GND #PWR03
+L GND #PWR15
 U 1 1 5399FE8D
 P 3800 6450
-F 0 "#PWR03" H 3800 6450 30  0001 C CNN
+F 0 "#PWR15" H 3800 6450 30  0001 C CNN
 F 1 "GND" H 3800 6380 30  0001 C CNN
 F 2 "" H 3800 6450 60  0000 C CNN
@@
 	1    0    0    -1
 $EndComp
-Text GLabel 3300 5650 0    60   Input ~ 12
+Text GLabel 1850 5650 0    60   Input ~ 12
 ICSPDAT
-Text GLabel 3400 5450 0    60   Input ~ 12
+Text GLabel 1850 5450 0    60   Input ~ 12
 VPP/MCLR
 Text GLabel 4450 1750 2    60   Input ~ 12
@@
 AUX
 $Comp
-L GND #PWR04
+L GND #PWR6
 U 1 1 539A0161
 P 4000 2550
-F 0 "#PWR04" H 4000 2550 30  0001 C CNN
+F 0 "#PWR6" H 4000 2550 30  0001 C CNN
 F 1 "GND" H 4000 2480 30  0001 C CNN
 F 2 "" H 4000 2550 60  0000 C CNN
@@
 ICSPCLK
 $Comp
-L PWR_FLAG #FLG05
+L PWR_FLAG #FLG1
 U 1 1 539A8F20
 P 1400 2100
-F 0 "#FLG05" H 1400 2195 30  0001 C CNN
+F 0 "#FLG1" H 1400 2195 30  0001 C CNN
 F 1 "PWR_FLAG" H 1400 2280 30  0000 C CNN
 F 2 "" H 1400 2100 60  0000 C CNN
@@
 $EndComp
 $Comp
-L PWR_FLAG #FLG06
+L PWR_FLAG #FLG2
 U 1 1 539A8F2F
 P 1750 2100
-F 0 "#FLG06" H 1750 2195 30  0001 C CNN
+F 0 "#FLG2" H 1750 2195 30  0001 C CNN
 F 1 "PWR_FLAG" H 1750 2280 30  0000 C CNN
 F 2 "" H 1750 2100 60  0000 C CNN
@@
 $EndComp
 $Comp
-L PWR_FLAG #FLG07
+L PWR_FLAG #FLG3
 U 1 1 539A8F3E
 P 2100 2100
-F 0 "#FLG07" H 2100 2195 30  0001 C CNN
+F 0 "#FLG3" H 2100 2195 30  0001 C CNN
 F 1 "PWR_FLAG" H 2100 2280 30  0000 C CNN
 F 2 "" H 2100 2100 60  0000 C CNN
@@
 $EndComp
 $Comp
-L VCC #PWR08
+L VCC #PWR3
 U 1 1 539A8F4B
 P 2100 2200
-F 0 "#PWR08" H 2100 2300 30  0001 C CNN
+F 0 "#PWR3" H 2100 2300 30  0001 C CNN
 F 1 "VCC" H 2100 2300 30  0000 C CNN
 F 2 "" H 2100 2200 60  0000 C CNN
@@
 $EndComp
 $Comp
-L GND #PWR09
+L GND #PWR4
 U 1 1 539A8F51
 P 1750 2250
-F 0 "#PWR09" H 1750 2250 30  0001 C CNN
+F 0 "#PWR4" H 1750 2250 30  0001 C CNN
 F 1 "GND" H 1750 2180 30  0001 C CNN
 F 2 "" H 1750 2250 60  0000 C CNN
@@
 $EndComp
 $Comp
-L +12V #PWR010
+L +12V #PWR2
 U 1 1 539A8F57
 P 1400 2200
-F 0 "#PWR010" H 1400 2150 20  0001 C CNN
+F 0 "#PWR2" H 1400 2150 20  0001 C CNN
 F 1 "+12V" H 1400 2300 30  0000 C CNN
 F 2 "" H 1400 2200 60  0000 C CNN
@@
 $EndComp
 $Comp
-L GND #PWR011
+L GND #PWR17
 U 1 1 54797D1B
 P 5900 6800
-F 0 "#PWR011" H 5900 6800 30  0001 C CNN
+F 0 "#PWR17" H 5900 6800 30  0001 C CNN
 F 1 "GND" H 5900 6730 30  0001 C CNN
 F 2 "" H 5900 6800 60  0000 C CNN
@@
 	3550 5250 3550 5450
 Wire Wire Line
-	3400 5450 4100 5450
+	1850 5450 4100 5450
 Wire Wire Line
 	4750 4500 4750 5000
@@
 	3800 6250 3800 6450
 Wire Wire Line
-	4100 5650 3300 5650
+	4100 5650 1850 5650
 Connection ~ 3550 5450
 Wire Wire Line
@@
 	6650 6150 6750 6150
 $Comp
-L GND #PWR012
+L GND #PWR18
 U 1 1 5479C839
 P 6650 6800
-F 0 "#PWR012" H 6650 6800 30  0001 C CNN
+F 0 "#PWR18" H 6650 6800 30  0001 C CNN
 F 1 "GND" H 6650 6730 30  0001 C CNN
 F 2 "" H 6650 6800 60  0000 C CNN
@@
 $EndComp
 $Comp
-L +12V #PWR013
+L +12V #PWR14
 U 1 1 5479C889
 P 8050 5300
-F 0 "#PWR013" H 8050 5250 20  0001 C CNN
+F 0 "#PWR14" H 8050 5250 20  0001 C CNN
 F 1 "+12V" H 8050 5400 30  0000 C CNN
 F 2 "" H 8050 5300 60  0000 C CNN
@@
 	8050 6250 7450 6250
 $Comp
-L GND #PWR014
+L GND #PWR19
 U 1 1 5479C910
 P 7600 6800
-F 0 "#PWR014" H 7600 6800 30  0001 C CNN
+F 0 "#PWR19" H 7600 6800 30  0001 C CNN
 F 1 "GND" H 7600 6730 30  0001 C CNN
 F 2 "" H 7600 6800 60  0000 C CNN
@@
 $EndComp
 $Comp
-L GND #PWR015
+L GND #PWR9
 U 1 1 5479CDA1
 P 3450 3850
-F 0 "#PWR015" H 3450 3850 30  0001 C CNN
+F 0 "#PWR9" H 3450 3850 30  0001 C CNN
 F 1 "GND" H 3450 3780 30  0001 C CNN
 F 2 "" H 3450 3850 60  0000 C CNN
@@
 $EndComp
 $Comp
-L +5V #PWR016
+L +5V #PWR12
 U 1 1 5479CDA9
 P 3550 4500
-F 0 "#PWR016" H 3550 4590 20  0001 C CNN
+F 0 "#PWR12" H 3550 4590 20  0001 C CNN
 F 1 "+5V" H 3550 4590 30  0000 C CNN
 F 2 "" H 3550 4500 60  0000 C CNN
@@
 	2850 3300 3050 3300
 $Comp
-L GND #PWR017
+L GND #PWR7
 U 1 1 5479CF78
 P 1850 3550
-F 0 "#PWR017" H 1850 3550 30  0001 C CNN
+F 0 "#PWR7" H 1850 3550 30  0001 C CNN
 F 1 "GND" H 1850 3480 30  0001 C CNN
 F 2 "" H 1850 3550 60  0000 C CNN
@@
 	3450 3850 3450 3600
 $Comp
-L PWR_FLAG #FLG018
+L PWR_FLAG #FLG4
 U 1 1 5479D2AB
 P 2450 2100
-F 0 "#FLG018" H 2450 2195 30  0001 C CNN
+F 0 "#FLG4" H 2450 2195 30  0001 C CNN
 F 1 "PWR_FLAG" H 2450 2280 30  0000 C CNN
 F 2 "" H 2450 2100 60  0000 C CNN
@@
 $EndComp
 $Comp
-L +5V #PWR019
+L +5V #PWR5
 U 1 1 5479D2B1
 P 2450 2250
-F 0 "#PWR019" H 2450 2340 20  0001 C CNN
+F 0 "#PWR5" H 2450 2340 20  0001 C CNN
 F 1 "+5V" H 2450 2340 30  0000 C CNN
 F 2 "" H 2450 2250 60  0000 C CNN
@@
 Wire Wire Line
 	1850 3400 1850 3550
-Wire Wire Line
-	1750 3200 1900 3200
-Wire Wire Line
-	1900 3200 1900 2950
-Wire Wire Line
-	1900 2950 7450 2950
-Wire Wire Line
-	7450 2950 7450 4350
 $Comp
 L RESISTOR R1
 U 1 1 5479D383
-P 7450 4500
-F 0 "R1" H 7600 4600 60  0000 C CNN
-F 1 "27K" H 7600 4450 60  0000 C CNN
-F 2 "~" H 7450 4500 60  0000 C CNN
-F 3 "~" H 7450 4500 60  0000 C CNN
-	1    7450 4500
-	1    0    0    -1
-$EndComp
-Wire Wire Line
-	7450 4650 7450 6150
-Text Notes 1950 2950 0    60   ~ 0
+P 2200 3800
+F 0 "R1" H 2350 3900 60  0000 C CNN
+F 1 "27K" H 2350 3750 60  0000 C CNN
+F 2 "~" H 2200 3800 60  0000 C CNN
+F 3 "~" H 2200 3800 60  0000 C CNN
+	1    2200 3800
+	1    0    0    -1
+$EndComp
+Text Notes 1850 3150 0    60   ~ 0
 12Vcc comandata
 $Comp
 L RESISTOR R2
 U 1 1 5479D629
-P 7150 5000
-F 0 "R2" H 7300 5100 60  0000 C CNN
-F 1 "100K" H 7300 4950 60  0000 C CNN
-F 2 "~" H 7150 5000 60  0000 C CNN
-F 3 "~" H 7150 5000 60  0000 C CNN
-	1    7150 5000
-	1    0    0    -1
-$EndComp
-$Comp
-L GND #PWR020
-U 1 1 5479D62F
-P 7150 5300
-F 0 "#PWR020" H 7150 5300 30  0001 C CNN
-F 1 "GND" H 7150 5230 30  0001 C CNN
-F 2 "" H 7150 5300 60  0000 C CNN
-F 3 "" H 7150 5300 60  0000 C CNN
-	1    7150 5300
-	1    0    0    -1
-$EndComp
-Wire Wire Line
-	7450 4750 7150 4750
-Wire Wire Line
-	7150 4750 7150 4850
-Connection ~ 7450 4750
-Wire Wire Line
-	7150 5300 7150 5150
-$Comp
-L GND #PWR021
+P 2200 4350
+F 0 "R2" H 2350 4450 60  0000 C CNN
+F 1 "100K" H 2350 4300 60  0000 C CNN
+F 2 "~" H 2200 4350 60  0000 C CNN
+F 3 "~" H 2200 4350 60  0000 C CNN
+	1    2200 4350
+	1    0    0    -1
+$EndComp
+$Comp
+L GND #PWR8
 U 1 1 5479D829
 P 2950 3850
-F 0 "#PWR021" H 2950 3850 30  0001 C CNN
+F 0 "#PWR8" H 2950 3850 30  0001 C CNN
 F 1 "GND" H 2950 3780 30  0001 C CNN
 F 2 "" H 2950 3850 60  0000 C CNN
@@
 Connection ~ 4400 3300
 $Comp
-L GND #PWR022
+L GND #PWR10
 U 1 1 5479DA5E
 P 4000 3850
-F 0 "#PWR022" H 4000 3850 30  0001 C CNN
+F 0 "#PWR10" H 4000 3850 30  0001 C CNN
 F 1 "GND" H 4000 3780 30  0001 C CNN
 F 2 "" H 4000 3850 60  0000 C CNN
@@
 $EndComp
 $Comp
-L GND #PWR023
+L GND #PWR11
 U 1 1 5479DA64
 P 4400 3850
-F 0 "#PWR023" H 4400 3850 30  0001 C CNN
+F 0 "#PWR11" H 4400 3850 30  0001 C CNN
 F 1 "GND" H 4400 3780 30  0001 C CNN
 F 2 "" H 4400 3850 60  0000 C CNN
@@
 Text Label 1800 3300 0    60   ~ 0
 +12V
+$Comp
+L GND #PWR13
+U 1 1 547B2460
+P 2200 4700
+F 0 "#PWR13" H 2200 4700 30  0001 C CNN
+F 1 "GND" H 2200 4630 30  0001 C CNN
+F 2 "" H 2200 4700 60  0000 C CNN
+F 3 "" H 2200 4700 60  0000 C CNN
+	1    2200 4700
+	1    0    0    -1
+$EndComp
+Wire Wire Line
+	1750 3200 2200 3200
+Wire Wire Line
+	2200 3200 2200 3650
+Wire Wire Line
+	2200 3950 2200 4200
+Wire Wire Line
+	2200 4500 2200 4700
+Wire Wire Line
+	2200 4050 2850 4050
+Wire Wire Line
+	2850 4050 2850 5650
+Connection ~ 2850 5650
+Connection ~ 2200 4050
+$Comp
+L PIC12F635_3 U2
+U 1 1 547B27DA
+P 4750 5950
+F 0 "U2" H 4500 6800 60  0000 C CNN
+F 1 "PIC12F635" H 5100 6800 60  0000 C CNN
+F 2 "~" H 4750 5950 60  0000 C CNN
+F 3 "~" H 4750 5950 60  0000 C CNN
+	1    4750 5950
+	1    0    0    -1
+$EndComp
 $EndSCHEMATC

Commit message: 2014-12-14 20:33 - commit with no comment
Parts:
- removed D4: DIODE, ~, symbol DIODE
- removed DL2: LED, ~, symbol LED
- removed R4: 470, ~, symbol RESISTOR
- removed U2: PIC12F635, ~, symbol PIC12F635_3
- added R3: 25K, ~, symbol RESISTOR
- added R5: 330, ~, symbol RESISTOR
- added U2: PIC12F635_4, ~, symbol PIC12F635_4
- C1, C3: value C -> 100nF
- C2: value CAPPOL -> 10uF
- R1: value 27K -> 4K7
- R2: value 100K -> 2K2
- R6: renamed from R5; value 470K -> 470
- renumbered DL3 to DL2, K1 to K2, R3 to R4
Connections:
- net labels added: +12Vcc CMD, +12Vcc \n(Autoradio), +5Vcc, OUT_LINE
- net labels removed: Out
- wire segments 63 -> 72
- no-connect marks 4 -> 2
Other:
- note added: "1"
- note added: "11"
- note added: "12"
- note added: "2"
- note added: "3.98 Volt"
- note added: "7"
- note added: "circa 5mA"
- note removed: "12Vcc comandata"
- moved on the sheet: C1, C3, D1, DL2, K2, P1, R1, R2, R4, R6, U1

Commit message: 2015-02-06 07:53 - commit with no comment
Parts:
- removed K2: 12Vcc, ~, symbol CONN_03
- removed K3: RELAY_1RT, ~, symbol RELAY_1RT
- removed P1: CONN_06, ~, symbol CONN_06
- removed R3: 25K, ~, symbol RESISTOR
- removed SW1: Power, ~, symbol PULSANTENC
- added C4: 10uF, ~, symbol CAPPOL
- added J1: 12Vcc, ~, symbol CONN_04
- added J2: ExtLED, ~, symbol CONN_02
- added J3: CONN_05, ~, symbol CONN_05
- added PB1: PButton, ~, symbol PULSANTENC
- added Q1: BC337-BC238, ~, symbol NPN
- added R1: 25K, ~, symbol RESISTOR
- added R7: 2k2, ~, symbol RESISTOR
- added RL1: RELAY_AUTORADIO, ~, symbol RELAY_AUTORADIO
- renumbered R1 to R2, R2 to R3
Connections:
- net labels added: +12V_CMD, +12Vcc (Autoradio), ClockOUT
- net labels removed: +12Vcc CMD, +12Vcc \n(Autoradio), +5Vcc, AUX
- wire segments 72 -> 82
Other:
- note removed: "1"
- note removed: "11"
- note removed: "12"
- note removed: "2"
- note removed: "7"
- moved on the sheet: D1, D2, DL1, DL2, IC1, R5
